File: PTP_Josip_Grgic_Project1/PTP_Josip_Grgic_Project1.kicad_sch (KiCad schematic)
At the start: 0 parts

Commit message: lv2
Parts:
- added C3: 22u, symbol Device:C_Polarized
- added C4: 1u, symbol Device:C
- added C6: 220u, symbol Device:C_Polarized
- added C7: 10u, symbol Device:C
- added C8: 100n, symbol Device:C
- added D1: 11DQ06, symbol Device:D_Schottky_Filled
- added D2, D3, D4, D5: ~, symbol Device:LED
- added J1: ~, symbol Connector:Screw_Terminal_01x02
- added L1: 330u, symbol Device:L
- added R1, R2: 2k, symbol Device:R
- added R3, R4: 47k, symbol Device:R
- added R6, R7, R8, R9: 4k7, symbol Device:R
- added SW1: ~, symbol Switch:SW_Push
- added SW2: ~, symbol Switch:SW_SPDT
- added U1: NE555P, Package_DIP:DIP-8_W7.62mm, symbol Timer:NE555P
- added U2: LM2574N-5, Package_DIP:DIP-8_W7.62mm, symbol Regulator_Switching:LM2574N-5
Connections:
- new net: C4.2, R1.1, R2.2, SW2.3 (A)
- new net: D5.1 (K), R9.1
- new net: C7.1, R4.2, U1.2 (TR), U1.6 (THR)
- new net: R3.2, R4.1, U1.7 (DIS)
- new net: R2.1, SW1.2
- new net: D1.1 (K), L1.1, U2.7 (OUT)
- new net: D3.1 (K), R7.1
- new net: D4.1 (K), R8.1
- new net: D2.1 (K), R6.1
- new net +5V: C6.1, C8.1, L1.2, R1.2, R3.1, U1.4 (R), U1.8 (VCC), U2.1 (FB)
- new net 555: SW2.2 (C), U1.3 (Q)
- new net Clock: SW2.1 (B)
- new net GND: C3.2, C4.1, C6.2, C7.2, C8.2, D1.2 (A), J1.1 (Pin_1), R6.2, R7.2, R8.2, R9.2, SW1.1, U1.1 (GND), U2.2 (SGND), U2.3 (~{ON}/OFF), U2.4 (PGND)
- new net Q0: D2.2 (A)
- new net Q1: D3.2 (A)
- new net Q2: D4.2 (A)
- new net Q3: D5.2 (A)
- new net VD: C3.1, J1.2 (Pin_2), U2.5 (VIN)
- no-connect marks 0 -> 1

Commit message: project1_lv3
Parts:
- removed C4: 1u, symbol Device:C
- removed R1, R2: 2k, symbol Device:R
- removed SW1: ~, symbol Switch:SW_Push
- removed SW2: ~, symbol Switch:SW_SPDT
- added C1: 1u, symbol Device:C
- added R5: 2k, symbol Device:R
- added R7: 10k, symbol Device:R
- added SW3: ~, symbol Switch:SW_Push
- added SW4: ~, symbol Switch:SW_SPDT
- added U3: ~, symbol SN74LVC1G11:SM74LVC1G11
- added U6: 74LVC1G11, symbol SN74LVC1G11:SM74LVC1G11
- renumbered C3 to C1, D2 to D1, D3 to D2, D4 to D3, D1 to D4, R6 to R1, R7 to R2, R8 to R3, R9 to R4
Connections:
- net +5V: now also R7.2, U6.5 (VCC)
- net 555: now also SW4.2 (C)
- net Clock: now also R7.1, SW4.1 (B), U6.6 (Input)
- net GND: now also C1.1, SW3.1, U6.2 (GND)
- net Q1: now also U6.1 (Input)
- net Q3: now also U6.3 (Input)
- new net: R5.1, SW3.2
- new net: C1.2, R5.2, SW4.3 (A)
Other:
- moved on the sheet: C1, C6, C7, C8, D1, D2, D3, D4, D5, J1, L1, R1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

Commit message: lv_4
lv4
Parts:
- removed U3: ~, symbol SN74LVC1G11:SM74LVC1G11
- added H1, H2, H3, H4: MountingHole, symbol Mechanical:MountingHole
- added R10, R11, R12, R15, R9: 10k, symbol Device:R
- added R14, R16, R17, R18, R5, R6, R8: 2k, symbol Device:R
- added U2, U3: 4027, symbol 4xxx:4027
- added U4: 74LS47, symbol 74xx:74LS47
- added U5: HDSP-7401, Display_7Segment:HDSP-7401, symbol Display_Character:HDSP-7401
- C1: footprint (none) -> Capacitor_THT:CP_Radial_D5.0mm_P2.00mm; Manufacture (none) -> AISHI; Manufacture part number  (none) -> EWH1EM220D11OT
- C2: renamed from C6; footprint (none) -> Capacitor_THT:CP_Radial_D5.0mm_P2.00mm; Manufacture (none) -> SAMWHA; Manufacture part number  (none) -> RD1A227M05011BB
- C3: renamed from C1; footprint (none) -> Capacitor_SMD:C_1206_3216Metric_Pad1.33x1.80mm_HandSolder; Manufacture (none) -> SAMSUNG; Manufacture part nmber  (none) -> CL31B105KBHNNNE
- C4: renamed from C8; footprint (none) -> Capacitor_SMD:C_1206_3216Metric_Pad1.33x1.80mm_HandSolder; Manufacture (none) -> SAMSUNG; Manufacture part number (none) -> CL31B104KBCNNNC
- C5: renamed from C7; footprint (none) -> Capacitor_SMD:C_1206_3216Metric_Pad1.33x1.80mm_HandSolder; Manufacture (none) -> SAMSUNG; Manufacture part number (none) -> CL31A106KBHNNNE
- U1: renamed from U2; footprint Package_DIP:DIP-8_W7.62mm -> Package_DIP:DIP-8_W7.62mm_Socket_LongPads; Manufacture (none) -> ONSEMI; Manufacture part number (none) -> LM2574N-5G
- renumbered R3 to R21, R4 to R22, R5 to R23, R7 to R24, U1 to U7
Connections:
- net +5V: now also R10.1, R11.1, R12.1, R15.1, R9.1, U2.16 (VDD), U3.16 (VDD), U4.16 (VCC), U5.1 (CA), U5.6 (CA)
- net Clock: now also U2.3 (C)
- net GND: now also U2.7 (S), U2.8 (VSS), U2.9 (S), U3.7 (S), U3.8 (VSS), U3.9 (S), U4.8 (GND)
- net Q0: now also U2.1 (Q), U2.13 (C), U4.7 (A)
- net Q1: now also U2.15 (Q), U3.3 (C), U4.1 (B)
- net Q2: now also U3.1 (Q), U3.13 (C), U4.2 (C)
- net Q3: now also U3.15 (Q), U4.6 (D)
- net Reset: now also U2.12 (R), U2.4 (R), U3.12 (R), U3.4 (R)
- new net: R10.2, U2.10 (J), U2.11 (K)
- new net: R6.1, U4.12 (b)
- new net: R6.2, U5.9 (B)
- new net: R12.2, U3.10 (J), U3.11 (K)
- new net: R14.1, U4.10 (d)
- new net: R8.1, U4.11 (c)
- new net: R5.1, U4.13 (a)
- new net: R18.1, U4.14 (g)
- new net: R17.1, U4.15 (f)
- new net: R15.2, U4.3 (LT), U4.4 (BI), U4.5 (RBI)
- new net: R16.1, U4.9 (e)
- new net: R11.2, U3.5 (K), U3.6 (J)
- new net: R9.2, U2.5 (K), U2.6 (J)
- new net: R5.2, U5.10 (A)
- new net: R17.2, U5.2 (F)
- new net: R18.2, U5.3 (G)
- new net: R16.2, U5.4 (E)
- new net: R14.2, U5.5 (D)
- new net: R8.2, U5.8 (C)
- no-connect marks 1 -> 6
Other:
- moved on the sheet: C3, C4, C5, D1, D2, D3, D5, R1, R2, R21, R22, R23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

Commit message: lv4_project
lv4
Parts:
- removed U6: 74LVC1G11, symbol SN74LVC1G11:SM74LVC1G11
- added U6: 74LVC1G11, Package_TO_SOT_SMD:SOT-23-6, symbol 74xGxx:74LVC1G11
- D1, D2, D3, D5: value ~ -> LED; footprint (none) -> LED_THT:LED_D5.0mm
- D4: footprint (none) -> Diode_THT:D_DO-41_SOD81_P12.70mm_Horizontal; Manufacture Part Number (none) -> 11DQ06TA; Manufacturer (none) -> SMC DIODE SOLUTIONS
- H1, H2, H3, H4: footprint (none) -> MountingHole:MountingHole_5.5mm
- J1: value ~ -> Screw_Terminal_01x02; footprint (none) -> TerminalBlock_MetzConnect:TerminalBlock_MetzConnect_Type011_RT05502HBLC_1x02_P5.00mm_Horizontal; Manufacturer (none) -> DEGSON ELECTRONICS; Manufacturer Part Number (none) -> DG301-5.0-02P-12-00A(H)
- L1: footprint (none) -> Inductor_THT:L_Radial_D7.2mm_P3.00mm_Murata_1700; Manufacturer (none) -> FERROCORE; Manufacturer Part Number  (none) -> COIL0608-0.33
- R1, R2, R3, R4: footprint (none) -> Resistor_THT:R_Axial_DIN0207_L6.3mm_D2.5mm_P10.16mm_Horizontal
- R10, R11, R12, R15, R9: footprint (none) -> Resistor_SMD:R_1206_3216Metric_Pad1.30x1.75mm_HandSolder
- R13: renamed from R23; footprint (none) -> Resistor_SMD:R_1206_3216Metric_Pad1.30x1.75mm_HandSolder; Manufacturer (none) -> ROYALOHM; Manufacturer Part Number (none) -> 1206S4F2001T5E
- R14, R16, R17, R18, R5, R6, R8: footprint (none) -> Resistor_SMD:R_1206_3216Metric_Pad1.30x1.75mm_HandSolder; Manufacturer (none) -> ROYALOHM; Manufacturer Part Number (none) -> 1206S4F2001T5E
- R19: renamed from R21; footprint (none) -> Resistor_SMD:R_1206_3216Metric_Pad1.30x1.75mm_HandSolder; Manufacturer (none) -> ROYALOHM; Manufacturer Part Number (none) -> 1206S4J0473T5E
- R20: renamed from R22; footprint (none) -> Resistor_SMD:R_1206_3216Metric_Pad1.30x1.75mm_HandSolder; Manufacturer (none) -> ROYALOHM; Manufacturer Part Number (none) -> 1206S4J0473T5E
- R7: renamed from R24; footprint (none) -> Resistor_SMD:R_1206_3216Metric_Pad1.30x1.75mm_HandSolder
- SW1: renamed from SW3; value ~ -> SW_Push; footprint (none) -> Button_Switch_THT:SW_PUSH_6mm_H4.3mm; Manufacturer (none) -> microswitch TACT; Manufacturer Part Number (none) -> TACT-64N-F
- SW2: renamed from SW4; footprint (none) -> Button_Switch_THT:SW_Slide_SPDT_Straight_CK_OS102011MS2Q; Manufacturer (none) -> C&K; Manufacturer Part Number (none) -> OS102011MS2QN1C
- U2, U3: footprint (none) -> Package_DIP:DIP-16_W7.62mm_Socket_LongPads; Manufacturer (none) -> RENESAS; Manufacturer Part Number (none) -> CD4027BMS
- U4: footprint (none) -> Package_DIP:DIP-16_W7.62mm_Socket_LongPads; Manufacturer (none) -> TEXAS INSTRUMENTS; Manufacturer Part Number (none) -> SN74LS47N
- U5: value HDSP-7401 -> FYS-3911BUHR-21; Manufacturer (none) -> FORYARD; Manufacturer Part Number (none) -> FYS-3911BUHR-21
- U7: Manufacturer (none) -> TEXAS INSTRUMENTS; Manufacturer Part Number (none) -> NE555P
Connections:
- net +5V: now also U6.5 (VCC)
- net Clock: now also U6.3
- net GND: now also U6.2 (GND)
- net Q1: now also U6.6
- net Q3: now also U6.1
- net Reset: now also U6.4
Other:
- note added: "555_timer"
- note added: "JK_bistabil"
- note added: "Led_diode"
- note added: "Montažne_rupe"
- note added: "Napajanje"
- note added: "Napajanje_bistabila"
- note added: "Reset_brojača"
- note added: "Tipkalo_i_ulaz_radnog_takta"
- moved on the sheet: D1, D2, D3, D5, R1, R2, R3, R4
