File: PTP_Josip_Grgic_Project1/PTP_Josip_Grgic_Project1.kicad_pcb (KiCad board)
At the start: 2 copper layers, 45 parts, among them J1 Screw_Terminal_01x02, SW1 SW_Push, U1 LM2574N-5, U2 4027, U3 4027, U4 74LS47, U5 FYS-3911BUHR-21, U6 74LVC1G11, U7 NE555P

Commit message: LV_7
Vjezba_7
Parts:
- moved R19 101.5 mm to (119.2, 91.5), turned to 90 degrees
- moved R20 100.5 mm to (119.2, 84.6), turned to 90 degrees
- moved U7 90.6 mm to (124.3, 84.2)
- moved C4 85.5 mm to (127.8, 95.8)
- moved C5 77.8 mm to (134.8, 86.6), turned to 90 degrees
- moved U5 75.8 mm to (204.7, 74.6)
- moved U6 64.0 mm to (148.1, 79.9)
- moved R17 58.3 mm to (198.0, 74.2)
- moved R18 58.3 mm to (197.8, 77.4)
- moved R16 54.9 mm to (198.3, 81.5)
- moved R6 53.9 mm to (198.3, 89.5)
- moved R14 53.6 mm to (198.4, 96.2)
- moved R8 53.6 mm to (198.4, 93.0)
- moved R5 53.3 mm to (198.4, 85.1)
- moved SW2 49.4 mm to (140.8, 77.3), turned to -90 degrees
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Routing:
- net GND: track 0.00 -> 156.2 mm, vias 0 -> 2
- net Clock: track 0.00 -> 50.0 mm
- net Net-(U7-DIS): track 0.00 -> 46.1 mm, vias 0 -> 2
- net +5V: track 0.00 -> 44.2 mm, vias 0 -> 2
- net Net-(D4-K): track 0.00 -> 42.0 mm, vias 0 -> 4
- net Net-(U2A-J): track 0.00 -> 40.8 mm
- net Net-(SW2-A): track 0.00 -> 38.5 mm
- net Q1: track 0.00 -> 36.1 mm, vias 0 -> 2
- net Q2: track 0.00 -> 34.6 mm, vias 0 -> 2
- net 555: track 0.00 -> 31.5 mm, vias 0 -> 4
- net Net-(U3A-J): track 0.00 -> 29.5 mm
- net Net-(U2B-J): track 0.00 -> 26.3 mm
- net Q0: track 0.00 -> 24.6 mm
- net Q3: track 0.00 -> 23.8 mm, vias 0 -> 4
- net VD: track 0.00 -> 21.1 mm
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- added copper zone on B.Cu, net GND
